Commit message: add cartographer and anvigation2

File: src/kkbot_description/urdf/kkbot.urdf.xacro (robot description, xacro)
@@ -32,5 +32,5 @@
         <xacro:cylinder_inertia m="0.2" r="${wheel_radius}" h="${wheel_length}" />
     </link>
-    <xacro:joint name="left_wheel" parent_name="base_link" type="continuous" origin_x="-0.02" origin_y="${bot_radius}" origin_z="-${bot_length / 2}" axis_x="0" axis_y="1" axis_z="0" />
+    <xacro:joint name="left_wheel" parent_name="base_link" type="continuous" origin_x="-0.05" origin_y="${bot_radius}" origin_z="-${bot_length / 2}" axis_x="0" axis_y="1" axis_z="0" />
     <!-- right_wheel -->
     <link name="right_wheel_link">
@@ -39,5 +39,5 @@
         <xacro:cylinder_inertia m="0.2" r="${wheel_radius}" h="${wheel_length}" />
     </link>
-    <xacro:joint name="right_wheel" parent_name="base_link" type="continuous" origin_x="-0.02" origin_y="-${bot_radius}" origin_z="-${bot_length / 2}" axis_x="0" axis_y="1" axis_z="0" />
+    <xacro:joint name="right_wheel" parent_name="base_link" type="continuous" origin_x="-0.05" origin_y="-${bot_radius}" origin_z="-${bot_length / 2}" axis_x="0" axis_y="1" axis_z="0" />
     <!-- caster -->
     <link name="caster_link">
@@ -47,3 +47,152 @@
     </link>
     <xacro:joint name="caster" parent_name="base_link" type="fixed" origin_x="0.06" origin_y="0" origin_z="-${bot_length / 2 + caster_radius}" axis_x="0" axis_y="1" axis_z="0" />
+    <!-- gazebo plugin -->
+    <gazebo>
+        <plugin name='diff_drive' filename='libgazebo_ros_diff_drive.so'>
+            <ros>
+                <namespace>/</namespace>
+                <remapping>cmd_vel:=cmd_vel</remapping>
+                <remapping>odom:=odom</remapping>
+            </ros>
+            <update_rate>30</update_rate>
+            <!-- wheels -->
+            <!-- <left_joint>left_wheel_joint</left_joint> -->
+            <!-- <right_joint>right_wheel_joint</right_joint> -->
+            <left_joint>left_wheel_joint</left_joint>
+            <right_joint>right_wheel_joint</right_joint>
+            <!-- kinematics -->
+            <wheel_separation>0.2</wheel_separation>
+            <wheel_diameter>0.065</wheel_diameter>
+            <!-- limits -->
+            <max_wheel_torque>20</max_wheel_torque>
+            <max_wheel_acceleration>1.0</max_wheel_acceleration>
+            <!-- output -->
+            <publish_odom>true</publish_odom>
+            <publish_odom_tf>true</publish_odom_tf>
+            <publish_wheel_tf>false</publish_wheel_tf>
+            <odometry_frame>odom</odometry_frame>
+            <robot_base_frame>base_footprint</robot_base_frame>
+        </plugin>
+                <plugin name="kkbot_joint_state" filename="libgazebo_ros_joint_state_publisher.so">
+            <ros>
+                <remapping>~/out:=joint_states</remapping>
+            </ros>
+            <update_rate>30</update_rate>
+            <joint_name>right_wheel_joint</joint_name>
+            <joint_name>left_wheel_joint</joint_name>
+        </plugin>
+    </gazebo>
+        <gazebo reference="imu_link">
+        <sensor name="imu_sensor" type="imu">
+            <plugin filename="libgazebo_ros_imu_sensor.so" name="imu_plugin">
+                <ros>
+                    <namespace>/</namespace>
+                    <remapping>~/out:=imu</remapping>
+                </ros>
+                <initial_orientation_as_reference>false</initial_orientation_as_reference>
+            </plugin>
+            <always_on>true</always_on>
+            <update_rate>100</update_rate>
+            <visualize>true</visualize>
+            <imu>
+                <angular_velocity>
+                    <x>
+                        <noise type="gaussian">
+                            <mean>0.0</mean>
+                            <stddev>2e-4</stddev>
+                            <bias_mean>0.0000075</bias_mean>
+                            <bias_stddev>0.0000008</bias_stddev>
+                        </noise>
+                    </x>
+                    <y>
+                        <noise type="gaussian">
+                            <mean>0.0</mean>
+                            <stddev>2e-4</stddev>
+                            <bias_mean>0.0000075</bias_mean>
+                            <bias_stddev>0.0000008</bias_stddev>
+                        </noise>
+                    </y>
+                    <z>
+                        <noise type="gaussian">
+                            <mean>0.0</mean>
+                            <stddev>2e-4</stddev>
+                            <bias_mean>0.0000075</bias_mean>
+                            <bias_stddev>0.0000008</bias_stddev>
+                        </noise>
+                    </z>
+                </angular_velocity>
+                <linear_acceleration>
+                    <x>
+                        <noise type="gaussian">
+                            <mean>0.0</mean>
+                            <stddev>1.7e-2</stddev>
+                            <bias_mean>0.1</bias_mean>
+                            <bias_stddev>0.001</bias_stddev>
+                        </noise>
+                    </x>
+                    <y>
+                        <noise type="gaussian">
+                            <mean>0.0</mean>
+                            <stddev>1.7e-2</stddev>
+                            <bias_mean>0.1</bias_mean>
+                            <bias_stddev>0.001</bias_stddev>
+                        </noise>
+                    </y>
+                    <z>
+                        <noise type="gaussian">
+                            <mean>0.0</mean>
+                            <stddev>1.7e-2</stddev>
+                            <bias_mean>0.1</bias_mean>
+                            <bias_stddev>0.001</bias_stddev>
+                        </noise>
+                    </z>
+                </linear_acceleration>
+            </imu>
+        </sensor>
+    </gazebo>
+    <gazebo reference="laser_link">
+        <material>Gazebo/Black</material>
+        <sensor name="laser_sensor" type="ray">
+            <always_on>true</always_on>
+            <visualize>true</visualize>
+            <update_rate>5</update_rate>
+            <pose>0 0 0.075 0 0 0</pose>
+            <ray>
+                <scan>
+                    <horizontal>
+                        <samples>360</samples>
+                        <resolution>1.000000</resolution>
+                        <min_angle>0.000000</min_angle>
+                        <max_angle>6.280000</max_angle>
+                    </horizontal>
+                </scan>
+                <range>
+                    <min>0.120000</min>
+                    <max>3.5</max>
+                    <resolution>0.015000</resolution>
+                </range>
+                <noise>
+                    <type>gaussian</type>
+                    <mean>0.0</mean>
+                    <stddev>0.01</stddev>
+                </noise>
+            </ray>
+            <plugin name="laserscan" filename="libgazebo_ros_ray_sensor.so">
+                <ros>
+                    <!-- <namespace>/tb3</namespace> -->
+                    <remapping>~/out:=scan</remapping>
+                </ros>
+                <output_type>sensor_msgs/LaserScan</output_type>
+                <frame_name>laser_link</frame_name>
+            </plugin>
+        </sensor>
+    </gazebo>
+    <gazebo reference="caster_link">
+        <material>Gazebo/Black</material>
+        <mu1 value="0.0"/>
+        <mu2 value="0.0"/>
+        <kp value="1000000.0"/>
+        <kd value="10.0"/>
+        <!-- <fdir1 value="0 0 1"/> -->
+    </gazebo>
 </robot>

File: src/kkbot_description/urdf/kkbot_base.urdf (robot description, URDF)
Before this commit: robot kkbot, 7 links, 6 joints
Joints:
- joint left_wheel_joint: origin xyz=-0.02 0.1 -0.06 -> xyz=-0.05 0.1 -0.06
- joint right_wheel_joint: origin xyz=-0.02 -0.1 -0.06 -> xyz=-0.05 -0.1 -0.06
